File: DC_MOTOR_0.1.kicad_sch (KiCad schematic)
At the start: 17 parts, among them P15 Pad, P17 Pad, U1 TLE9201SG

Commit message: update
Parts:
- C1, C10, C2, C3, C4, C5, C6, C7, C8, C9: footprint hellen-one-common:C0805 -> kicad6-libraries:C0805
- C11, C12, C13: footprint hellen-one-common:C0603 -> kicad6-libraries:C0603
- P15, P17: footprint hellen-one-common:PAD-TH -> kicad6-libraries:PAD-TH
- R9: footprint hellen-one-common:R0603 -> kicad6-libraries:R0603
Changed lines of the file:
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@@
 			)
 		)
-		(property "Footprint" "hellen-one-common:C0805"
+		(property "Footprint" "kicad6-libraries:C0805"
 			(at 148.59 86.36 0)
 			(effects
@@
 			)
 		)
-		(property "Footprint" "hellen-one-common:C0805"
+		(property "Footprint" "kicad6-libraries:C0805"
 			(at 121.92 86.36 0)
 			(effects
@@
 			)
 		)
-		(property "Footprint" "hellen-one-common:C0805"
+		(property "Footprint" "kicad6-libraries:C0805"
 			(at 113.03 86.36 0)
 			(effects
@@
 			)
 		)
-		(property "Footprint" "hellen-one-common:R0603"
+		(property "Footprint" "kicad6-libraries:R0603"
 			(at 223.52 95.25 0)
 			(effects
@@
 			)
 		)
-		(property "Footprint" "hellen-one-common:C0805"
+		(property "Footprint" "kicad6-libraries:C0805"
 			(at 95.25 86.36 0)
 			(effects
@@
 			)
 		)
-		(property "Footprint" "hellen-one-common:C0805"
+		(property "Footprint" "kicad6-libraries:C0805"
 			(at 104.14 86.36 0)
 			(effects
@@
 			)
 		)
-		(property "Footprint" "hellen-one-common:C0805"
+		(property "Footprint" "kicad6-libraries:C0805"
 			(at 77.47 86.36 0)
 			(effects
@@
 			)
 		)
-		(property "Footprint" "hellen-one-common:C0603"
+		(property "Footprint" "kicad6-libraries:C0603"
 			(at 166.37 86.36 0)
 			(effects
@@
 			)
 		)
-		(property "Footprint" "hellen-one-common:C0805"
+		(property "Footprint" "kicad6-libraries:C0805"
 			(at 157.48 86.36 0)
 			(effects
@@
 			)
 		)
-		(property "Footprint" "hellen-one-common:C0805"
+		(property "Footprint" "kicad6-libraries:C0805"
 			(at 139.7 86.36 0)
 			(effects
@@
 			)
 		)
-		(property "Footprint" "hellen-one-common:PAD-TH"
+		(property "Footprint" "kicad6-libraries:PAD-TH"
 			(at 220.98 111.76 0)
 			(effects
@@
 			)
 		)
-		(property "Footprint" "hellen-one-common:C0805"
+		(property "Footprint" "kicad6-libraries:C0805"
 			(at 130.81 86.36 0)
 			(effects
@@
 			)
 		)
-		(property "Footprint" "hellen-one-common:C0805"
+		(property "Footprint" "kicad6-libraries:C0805"
 			(at 86.36 86.36 0)
 			(effects
@@
 			)
 		)
-		(property "Footprint" "hellen-one-common:C0603"
+		(property "Footprint" "kicad6-libraries:C0603"
 			(at 179.07 90.17 0)
 			(effects
@@
 			)
 		)
-		(property "Footprint" "hellen-one-common:C0603"
+		(property "Footprint" "kicad6-libraries:C0603"
 			(at 179.07 114.3 0)
 			(effects
@@
 			)
 		)
-		(property "Footprint" "hellen-one-common:PAD-TH"
+		(property "Footprint" "kicad6-libraries:PAD-TH"
 			(at 220.98 109.22 0)
 			(effects
