File: IGN6.kicad_sch (KiCad schematic)
At the start: 16 parts, among them Q10 ISL9V3040D3ST, Q7 ISL9V3040D3ST, Q8 ISL9V3040D3ST, Q9 ISL9V3040D3ST

Commit message: update
Parts:
- R17, R18, R19, R23: footprint hellen-one-common:R0603 -> kicad6-libraries:R0603
Changed lines of the file:
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@@
 			)
 		)
-		(property "Footprint" "hellen-one-common:R0603"
+		(property "Footprint" "kicad6-libraries:R0603"
 			(at 129.54 66.04 0)
 			(effects
@@
 			)
 		)
-		(property "Footprint" "hellen-one-common:R0603"
+		(property "Footprint" "kicad6-libraries:R0603"
 			(at 129.54 93.98 0)
 			(effects
@@
 			)
 		)
-		(property "Footprint" "hellen-one-common:R0603"
+		(property "Footprint" "kicad6-libraries:R0603"
 			(at 176.53 93.98 0)
 			(effects
@@
 			)
 		)
-		(property "Footprint" "hellen-one-common:R0603"
+		(property "Footprint" "kicad6-libraries:R0603"
 			(at 176.53 66.04 0)
 			(effects
