File: INJ6.kicad_sch (KiCad schematic)
At the start: 6 parts, among them U10 VNLD5160TR-E, U9 VNLD5160TR-E

Commit message: update
Parts:
- R29, R30, R31, R32: footprint hellen-one-common:R0603 -> kicad6-libraries:R0603
Changed lines of the file:
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@@
 			)
 		)
-		(property "Footprint" "hellen-one-common:R0603"
+		(property "Footprint" "kicad6-libraries:R0603"
 			(at 170.18 76.2 0)
 			(effects
@@
 			)
 		)
-		(property "Footprint" "hellen-one-common:R0603"
+		(property "Footprint" "kicad6-libraries:R0603"
 			(at 193.04 97.79 0)
 			(effects
@@
 			)
 		)
-		(property "Footprint" "hellen-one-common:R0603"
+		(property "Footprint" "kicad6-libraries:R0603"
 			(at 193.04 71.12 0)
 			(effects
@@
 			)
 		)
-		(property "Footprint" "hellen-one-common:R0603"
+		(property "Footprint" "kicad6-libraries:R0603"
 			(at 170.18 102.87 0)
 			(effects
