File: LS4.kicad_sch (KiCad schematic)
At the start: 6 parts, among them U7 VNLD5160TR-E, U8 VNLD5160TR-E

Commit message: update
Parts:
- R10, R11, R12, R13: footprint hellen-one-common:R0603 -> kicad6-libraries:R0603
Changed lines of the file:
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@@
 			)
 		)
-		(property "Footprint" "hellen-one-common:R0603"
+		(property "Footprint" "kicad6-libraries:R0603"
 			(at 200.66 91.44 0)
 			(effects
@@
 			)
 		)
-		(property "Footprint" "hellen-one-common:R0603"
+		(property "Footprint" "kicad6-libraries:R0603"
 			(at 200.66 118.11 0)
 			(effects
@@
 			)
 		)
-		(property "Footprint" "hellen-one-common:R0603"
+		(property "Footprint" "kicad6-libraries:R0603"
 			(at 175.26 123.19 0)
 			(effects
@@
 			)
 		)
-		(property "Footprint" "hellen-one-common:R0603"
+		(property "Footprint" "kicad6-libraries:R0603"
 			(at 175.26 96.52 0)
 			(effects
