File: LS_HOT.kicad_sch (KiCad schematic)
At the start: 3 parts, among them U6 VNLD5160TR-E

Commit message: update
Parts:
- R15, R16: footprint hellen-one-common:R0603 -> kicad6-libraries:R0603
Changed lines of the file:
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@@
 			)
 		)
-		(property "Footprint" "hellen-one-common:R0603"
+		(property "Footprint" "kicad6-libraries:R0603"
 			(at 184.15 90.17 0)
 			(effects
@@
 			)
 		)
-		(property "Footprint" "hellen-one-common:R0603"
+		(property "Footprint" "kicad6-libraries:R0603"
 			(at 172.72 95.25 0)
 			(effects
