File: MAP.kicad_sch (KiCad schematic)
At the start: 2 parts, among them U3 MPX4/MPXH6400_MAP

Commit message: update
Parts:
- C27: footprint hellen-one-common:C0603 -> kicad6-libraries:C0603
Changed lines of the file:
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@@
 			)
 		)
-		(property "Footprint" "hellen-one-common:C0603"
+		(property "Footprint" "kicad6-libraries:C0603"
 			(at 161.29 95.25 0)
 			(effects
