File: egt.kicad_sch (KiCad schematic)
At the start: 9 parts, among them U4 MAX31855KASA

Commit message: update
Parts:
- C28, C29, C30, C31, C32: footprint hellen-one-common:C0603 -> kicad6-libraries:C0603
Changed lines of the file:
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@@
 			)
 		)
-		(property "Footprint" "hellen-one-common:C0603"
+		(property "Footprint" "kicad6-libraries:C0603"
 			(at 139.7 104.14 0)
 			(effects
@@
 			)
 		)
-		(property "Footprint" "hellen-one-common:C0603"
+		(property "Footprint" "kicad6-libraries:C0603"
 			(at 193.04 76.2 0)
 			(effects
@@
 			)
 		)
-		(property "Footprint" "hellen-one-common:C0603"
+		(property "Footprint" "kicad6-libraries:C0603"
 			(at 154.94 104.14 0)
 			(effects
@@
 			)
 		)
-		(property "Footprint" "hellen-one-common:C0603"
+		(property "Footprint" "kicad6-libraries:C0603"
 			(at 180.34 76.2 0)
 			(effects
@@
 			)
 		)
-		(property "Footprint" "hellen-one-common:C0603"
+		(property "Footprint" "kicad6-libraries:C0603"
 			(at 146.05 93.98 0)
 			(effects
